File: kicad/system_LED.kicad_sch (KiCad schematic)
At the start: 3 parts

Commit message: fix: change R fp to a smaller one
Signed-off-by: Bobo Bäck Engström <bobo@id8-engineering.io>
Parts:
- R14: footprint seven-lib:R_0603_1608Metric -> seven-lib:R_0402_1005Metric
Changed lines of the file:
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@@
 			)
 		)
-		(property "Footprint" "seven-lib:R_0603_1608Metric"
+		(property "Footprint" "seven-lib:R_0402_1005Metric"
 			(at 77.47 86.868 90)
 			(effects
