File: kicad/system_LED.kicad_sch (KiCad schematic)
At the start: 3 parts

Commit message: fix: changes made according to review meeting
Signed-off-by: Bobo Bäck Engström <bobo@id8-engineering.io>
Parts:
- added TP5: SYSTEM_LED, seven-lib:TestPoint_Pad_2.0x2.0mm, symbol seven_lib:TestPoint
Connections:
- net at D5.3 (DIN), R14.2: now also TP5.1
Changed lines of the file:
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@@
+		(color 0 0 0 0)
+	)
+	(junction
+		(at 83.82 85.09)
+		(diameter 0)
 		(color 0 0 0 0)
 	)
@@
 	(wire
 		(pts
-			(xy 81.28 85.09) (xy 86.36 85.09)
+			(xy 83.82 90.17) (xy 83.82 85.09)
+		)
+		(stroke
+			(width 0)
+			(type default)
+		)
+	)
+	(wire
+		(pts
+			(xy 81.28 85.09) (xy 83.82 85.09)
 		)
 		(stroke
@@
 		(pts
 			(xy 96.52 71.12) (xy 93.98 71.12)
+		)
+		(stroke
+			(width 0)
+			(type default)
+		)
+	)
+	(wire
+		(pts
+			(xy 83.82 85.09) (xy 86.36 85.09)
 		)
 		(stroke
@@
 					(unit 1)
 				)
+			)
+		)
+	)
+	(symbol
+		(lib_id "seven_lib:TestPoint")
+		(at 83.82 90.17 180)
+		(unit 1)
+		(exclude_from_sim no)
+		(in_bom yes)
+		(on_board yes)
+		(dnp no)
+		(property "Reference" "TP5"
+			(at 79.883 92.075 0)
+			(effects
+				(font
+					(size 1.27 1.27)
+				)
+			)
+		)
+		(property "Value" "SYSTEM_LED"
+			(at 79.883 94.615 0)
+			(effects
+				(font
+					(size 1.27 1.27)
+				)
+			)
+		)
+		(property "Footprint" "seven-lib:TestPoint_Pad_2.0x2.0mm"
+			(at 78.74 90.17 0)
+			(effects
+				(font
+					(size 1.27 1.27)
+				)
+				(hide yes)
+			)
+		)
+		(property "Datasheet" "~"
+			(at 78.74 90.17 0)
+			(effects
+				(font
+					(size 1.27 1.27)
+				)
+				(hide yes)
+			)
+		)
+		(property "Description" "test point"
+			(at 83.82 90.17 0)
+			(effects
+				(font
+					(size 1.27 1.27)
+				)
+				(hide yes)
+			)
+		)
+		(pin "1"
+		)
+		(instances
+			(project "seven"
+				(path "/8e3cc843-5797-49f3-8b3a-1c11450ccd1e/57402695-b5b6-411c-ba67-6244479e2395"
+					(reference "TP5")
+					(unit 1)
+				)

Commit message: feat(PCB): set component-placement example on PCB
This pr will fail due to DRC, skip this and lets have a conversation
about the placement only

Signed-off-by: Bobo Bäck Engström <bobo@id8-engineering.io>
Parts:
- removed TP5: SYSTEM_LED, seven-lib:TestPoint_Pad_2.0x2.0mm, symbol seven_lib:TestPoint
- C20: MPN (none) -> GRM155R71C104KA88D
- D5: MPN (none) -> SK6805-EC15
- R14: MPN (none) -> RC0402FR-07220RL
