File: kicad/power_supply.kicad_sch (KiCad schematic)
At the start: 15 parts, among them J5 Conn_01x02, U5 ISL85410FRZ-T7A

Commit message: fix: make changes according to ID8 review meeting
Signed-off-by: Bobo Bäck Engström <bobo@id8-engineering.io>
Connections:
- net EN: now reaches C32.1, J5.2 (VIN), U5.4 (VIN), U5.7 (EN)
Other:
- moved on the sheet: C32
Changed lines of the file:
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@@
+	)
+	(junction
+		(at 35.56 83.82)
+		(diameter 0)
+		(color 0 0 0 0)
+	)
+	(junction
+		(at 158.75 74.93)
+		(diameter 0)
+		(color 0 0 0 0)
+	)
+	(junction
+		(at 62.23 87.63)
+		(diameter 0)
+		(color 0 0 0 0)
+	)
+	(junction
+		(at 53.34 104.14)
+		(diameter 0)
+		(color 0 0 0 0)
 	)
 	(junction
@@
 	)
 	(junction
-		(at 58.42 87.63)
-		(diameter 0)
-		(color 0 0 0 0)
-	)
-	(junction
-		(at 53.34 105.41)
-		(diameter 0)
-		(color 0 0 0 0)
-	)
-	(junction
-		(at 35.56 83.82)
-		(diameter 0)
-		(color 0 0 0 0)
-	)
-	(junction
 		(at 35.56 90.17)
 		(diameter 0)
 		(color 0 0 0 0)
 	)
-	(junction
-		(at 158.75 74.93)
-		(diameter 0)
-		(color 0 0 0 0)
-	)
 	(no_connect
 		(at 67.31 82.55)
@@
 	(wire
 		(pts
-			(xy 107.95 105.41) (xy 107.95 95.25)
+			(xy 62.23 87.63) (xy 67.31 87.63)
 		)
 		(stroke
@@
 		)
 	)
-	(wire
-		(pts
-			(xy 53.34 87.63) (xy 53.34 105.41)
-		)
-		(stroke
-			(width 0)
-			(type default)
-		)
-	)
 	(polyline
 		(pts
@@
 	(wire
 		(pts
-			(xy 58.42 87.63) (xy 67.31 87.63)
-		)
-		(stroke
-			(width 0)
-			(type default)
-		)
-	)
-	(wire
-		(pts
-			(xy 53.34 105.41) (xy 107.95 105.41)
-		)
-		(stroke
-			(width 0)
-			(type default)
-		)
-	)
-	(wire
-		(pts
-			(xy 58.42 101.6) (xy 62.23 101.6)
-		)
-		(stroke
-			(width 0)
-			(type default)
-		)
-	)
-	(wire
-		(pts
-			(xy 35.56 62.23) (xy 35.56 83.82)
+			(xy 53.34 104.14) (xy 53.34 109.22)
 		)
 		(stroke
@@
 	(wire
 		(pts
+			(xy 48.26 104.14) (xy 53.34 104.14)
+		)
+		(stroke
+			(width 0)
+			(type default)
+		)
+	)
+	(wire
+		(pts
 			(xy 30.48 83.82) (xy 35.56 83.82)
 		)
@@
 	(wire
 		(pts
+			(xy 35.56 55.88) (xy 35.56 83.82)
+		)
+		(stroke
+			(width 0)
+			(type default)
+		)
+	)
+	(wire
+		(pts
 			(xy 158.75 85.09) (xy 158.75 87.63)
 		)
@@
 	(wire
 		(pts
-			(xy 53.34 105.41) (xy 53.34 109.22)
+			(xy 158.75 55.88) (xy 158.75 74.93)
 		)
 		(stroke
@@
 	(wire
 		(pts
-			(xy 35.56 62.23) (xy 158.75 62.23)
+			(xy 35.56 55.88) (xy 158.75 55.88)
 		)
 		(stroke
@@
 	(wire
 		(pts
+			(xy 53.34 87.63) (xy 62.23 87.63)
+		)
+		(stroke
+			(width 0)
+			(type default)
+		)
+	)
+	(wire
+		(pts
 			(xy 59.69 77.47) (xy 59.69 80.01)
 		)
@@
 	(wire
 		(pts
-			(xy 53.34 87.63) (xy 58.42 87.63)
-		)
-		(stroke
-			(width 0)
-			(type default)
-		)
-	)
-	(wire
-		(pts
 			(xy 62.23 101.6) (xy 62.23 109.22)
 		)
@@
 	(wire
 		(pts
-			(xy 158.75 62.23) (xy 158.75 74.93)
-		)
-		(stroke
-			(width 0)
-			(type default)
-		)
-	)
-	(wire
-		(pts
 			(xy 24.13 90.17) (xy 24.13 95.25)
 		)
@@
 	(wire
 		(pts
-			(xy 58.42 99.06) (xy 58.42 101.6)
+			(xy 62.23 99.06) (xy 62.23 101.6)
+		)
+		(stroke
+			(width 0)
+			(type default)
+		)
+	)
+	(wire
+		(pts
+			(xy 53.34 87.63) (xy 53.34 104.14)
 		)
 		(stroke
@@
 	(wire
 		(pts
-			(xy 58.42 87.63) (xy 58.42 91.44)
+			(xy 110.49 95.25) (xy 107.95 95.25)
+		)
+		(stroke
+			(width 0)
+			(type default)
+		)
+	)
+	(wire
+		(pts
+			(xy 62.23 87.63) (xy 62.23 91.44)
 		)
 		(stroke
@@
 			(width 0)
 			(type default)
+		)
+	)
+	(label "EN"
+		(at 110.49 95.25 0)
+		(effects
+			(font
+				(size 1.27 1.27)
+			)
+			(justify left bottom)
+		)
+	)
+	(label "EN"
+		(at 48.26 104.14 0)
+		(effects
+			(font
+				(size 1.27 1.27)
+			)
+			(justify left bottom)
 		)
 	)
@@
 	(symbol
 		(lib_id "seven_lib:C")
-		(at 58.42 95.25 0)
-		(unit 1)
-		(exclude_from_sim no)
-		(in_bom yes)
-		(on_board yes)
-		(dnp no)
-		(fields_autoplaced yes)
+		(at 62.23 95.25 0)
+		(unit 1)
+		(exclude_from_sim no)
+		(in_bom yes)
+		(on_board yes)
+		(dnp no)
 		(property "Reference" "C32"
-			(at 62.23 93.9799 0)
+			(at 62.23 93.218 0)
 			(effects
 				(font
@@
 		)
 		(property "Value" "10uF"
-			(at 62.23 96.5199 0)
+			(at 62.23 97.79 0)
 			(effects
 				(font
@@
 		)
 		(property "Footprint" "seven-lib:C_1812_4532Metric"
-			(at 59.3852 99.06 0)
+			(at 63.1952 99.06 0)
 			(effects
 				(font
@@
 		)
 		(property "Datasheet" "~"
-			(at 58.42 95.25 0)
+			(at 62.23 95.25 0)
 			(effects
 				(font
@@
 		)
 		(property "Description" "Unpolarized capacitor"
-			(at 58.42 95.25 0)
-			(effects
-				(font
+			(at 62.23 95.25 0)
+			(effects
+				(font
