File: kicad/PMIC.kicad_sch (KiCad schematic)
At the start: 25 parts, among them U4 nPM1300-QEXX

Commit message: feat: Update for 0.3.0 release
Add power rail controlled by PMIC load switch.
Change location for testpads to be cleaner
remove TC2030 and add JST connector for RPI debug probe
remove VDD_GPIO jumper
fix silkscreen

Signed-off-by: Bobob Bäck Engström <bobo@id8-engineering.io>
Parts:
- removed D2: BAT54KFILM, seven-lib:D_SOD-523, symbol seven_lib:BAT54W
- removed R9: 0, seven-lib:R_0402_1005Metric, symbol seven_lib:R
- added JP3, JP4: SolderJumper_2_Bridged, seven-lib:SolderJumper-2_P1.3mm_Bridged_RoundedPad1.0x1.5mm, symbol seven_lib:SolderJumper_2_Bridged
- renumbered TP18 to VDD_1V8, TP20 to VDD_3V3, TP19 to VDD_GNSS1
Connections:
- net GND: no longer U4.30 (LSIN2/VINLDO2), U4.31 (LSOUT2/VOUTLDO2)
- net VDD_1V8: no longer C4.1, R17.2, R18.2, U4.12 (VDDIO)
- net VDD_3V3: now also C4.1, R17.2, R18.2, U4.12 (VDDIO), U4.30 (LSIN2/VINLDO2), JP3.2 (B), JP4.2 (B)
- net VDD_GNSS: now also JP3.1 (A)
- new net VDD_POWER_LED: JP4.1 (A), U4.31 (LSOUT2/VOUTLDO2)
Other:
- moved on the sheet: VDD_GNSS1
