File: kicad/JST-SH.kicad_sch (KiCad schematic)
At the start: 1 part, among them J1 JST_SH_BM03B-SRSS-TB_1x03

Commit message: feat: Update for 0.3.0 release
Add power rail controlled by PMIC load switch.
Change location for testpads to be cleaner
remove TC2030 and add JST connector for RPI debug probe
remove VDD_GPIO jumper
fix silkscreen

Signed-off-by: Bobob Bäck Engström <bobo@id8-engineering.io>
Changed lines of the file:
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@@
 		)
 	)
-	(text_box "This circuit provides a Tag-Connect TC2030 programming and debugging interface for the MCU. It exposes the SWD (Serial Wire Debug) signals and power reference required to program and debug the device."
+	(text_box "FLASH CONNECTOR ONLY\nJST-SH operating rating: -25°C to +85°C.\nNot required for normal board operation.\nDo not connect, disconnect, or use this interface below -25°C."
 		(exclude_from_sim no)
 		(at 176.53 24.13 0)
@@
 		)
 	)
-	(text_box "JTAG SWD TC2030"
+	(text_box "JST-SH SWD Connector\n"
 		(exclude_from_sim no)
 		(at 176.53 12.7 0)

Commit message: fix: swap swclk and swdio for jst-sh contact
Signed-off-by: Bobob Bäck Engström <bobo@id8-engineering.io>
Connections:
- net SWCLK: now also J1.1 (SWCLK); no longer J1.3 (SWCLK)
- net SWDIO: now also J1.3 (SWDIO); no longer J1.1 (SWDIO)
Changed lines of the file:
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@@
 	(hierarchical_label "SWDIO"
 		(shape bidirectional)
-		(at 81.28 82.55 180)
+		(at 81.28 87.63 180)
 		(effects
 			(font
@@
 	(hierarchical_label "SWCLK"
 		(shape output)
-		(at 81.28 87.63 180)
+		(at 81.28 82.55 180)
 		(effects
 			(font
